Commit message: Fixed fetch urdf parsing

File: include/test_urdf/fetch.urdf (robot description, URDF)
Before this commit: robot fetch_arm_no_helpers, 9 links, 8 joints
Links:
- removed link arm_mount_link
- removed link ee_link
- added link base_link, mass 70.1294; collision mesh filename=package://meshes/base_link_collision.STL; visual mesh filename=package://meshes/base_link.dae
- added link estop_link, mass 0.00196130439134723; visual mesh filename=package://meshes/estop_link.dae
- added link gripper_link, mass 1.5175; collision mesh filename=package://meshes/gripper_link.STL; visual mesh filename=package://meshes/gripper_link.dae
- added link head_camera_depth_frame
- added link head_camera_depth_optical_frame
- added link head_camera_link
- added link head_camera_rgb_frame
- added link head_camera_rgb_optical_frame
- added link head_pan_link, mass 2.2556; collision mesh filename=package://meshes/head_pan_link_collision.STL; visual mesh filename=package://meshes/head_pan_link.dae
- added link head_tilt_link, mass 0.9087; collision mesh filename=package://meshes/head_tilt_link_collision.STL; visual mesh filename=package://meshes/head_tilt_link.dae
- added link l_gripper_finger_link, mass 0.0798; collision mesh filename=package://meshes/l_gripper_finger_link.STL; visual mesh filename=package://meshes/l_gripper_finger_link.STL
- added link r_gripper_finger_link, mass 0.0798; collision mesh filename=package://meshes/r_gripper_finger_link.STL; visual mesh filename=package://meshes/r_gripper_finger_link.STL
- added link torso_fixed_link, mass 13.2775; collision mesh filename=package://meshes/torso_fixed_link.STL; visual mesh filename=package://meshes/torso_fixed_link.dae
- added link torso_lift_link, mass 10.7796; collision mesh filename=package://meshes/torso_lift_link_collision.STL; visual mesh filename=package://meshes/torso_lift_link.dae
- link elbow_flex_link: geometry collision mesh filename=package://meshes/elbow_flex_link_collision.STL; visual mesh filename=package://meshes/elbow_flex_link.dae
- link forearm_roll_link: geometry collision mesh filename=package://meshes/forearm_roll_link_collision.STL; visual mesh filename=package://meshes/forearm_roll_link.dae
- link shoulder_lift_link: geometry collision mesh filename=package://meshes/shoulder_lift_link_collision.STL; visual mesh filename=package://meshes/shoulder_lift_link.dae
- link shoulder_pan_link: geometry collision mesh filename=package://meshes/shoulder_pan_link_collision.STL; visual mesh filename=package://meshes/shoulder_pan_link.dae
- link upperarm_roll_link: geometry collision mesh filename=package://meshes/upperarm_roll_link_collision.STL; visual mesh filename=package://meshes/upperarm_roll_link.dae
- link wrist_flex_link: geometry collision mesh filename=package://meshes/wrist_flex_link_collision.STL; visual mesh filename=package://meshes/wrist_flex_link.dae
- link wrist_roll_link: geometry collision mesh filename=package://meshes/wrist_roll_link_collision.STL; visual mesh filename=package://meshes/wrist_roll_link.dae
Joints:
- removed joint ee_fixed
- added joint estop_joint: type fixed, parent base_link, child estop_link, origin xyz=-0.12465 0.23892 0.31127 rpy=1.5708 0 0, axis 0 0 0
- added joint gripper_axis: type fixed, parent wrist_roll_link, child gripper_link, origin xyz=0.16645 0 0 rpy=0 0 0, axis 0 1 0
- added joint head_camera_depth_joint: type fixed, parent head_camera_link, child head_camera_depth_frame, origin xyz=0 0.045 0 rpy=0 0 0
- added joint head_camera_depth_optical_joint: type fixed, parent head_camera_depth_frame, child head_camera_depth_optical_frame, origin xyz=0 0 0 rpy=-1.57079632679 0 -1.57079632679
- added joint head_camera_joint: type fixed, parent head_tilt_link, child head_camera_link, origin xyz=0.055 0 0.0225 rpy=0 0 0
- added joint head_camera_rgb_joint: type fixed, parent head_camera_link, child head_camera_rgb_frame, origin xyz=0 0.02 0 rpy=0 0 0
- added joint head_camera_rgb_optical_joint: type fixed, parent head_camera_rgb_frame, child head_camera_rgb_optical_frame, origin xyz=0 0 0 rpy=-1.57079632679 0 -1.57079632679
- added joint head_pan_joint: type fixed, parent torso_lift_link, child head_pan_link, origin xyz=0.053125 0 0.603001417713939 rpy=0 0 0, axis 0 0 1
- added joint head_tilt_joint: type fixed, parent head_pan_link, child head_tilt_link, origin xyz=0.14253 0 0.057999 rpy=0 0 0, axis 0 1 0
- added joint l_gripper_finger_joint: type fixed, parent gripper_link, child l_gripper_finger_link, origin xyz=0 -0.065425 0 rpy=0 0 0, axis 0 -1 0
- added joint r_gripper_finger_joint: type fixed, parent gripper_link, child r_gripper_finger_link, origin xyz=0 0.065425 0 rpy=0 0 0, axis 0 1 0
- added joint torso_fixed_joint: type fixed, parent base_link, child torso_fixed_link, origin xyz=-0.086875 0 0.377425 rpy=-6.12303176911189E-17 0 0, axis 0 1 0
- added joint torso_lift_joint: type prismatic, parent base_link, child torso_lift_link, origin xyz=-0.086875 0 0.37743 rpy=-6.123E-17 0 0, axis 0 0 1, limit lower=0 upper=0.38615 effort=450.0 velocity=0.1
- joint elbow_flex_joint: axis 0 0 1 -> 0 1 0
- joint forearm_roll_joint: axis 0 0 1 -> 1 0 0
- joint shoulder_lift_joint: axis 0 0 1 -> 0 1 0; origin xyz=0.117 0 0.06 rpy=0 0 0 -> xyz=0.117 0 0.0599999999999999 rpy=0 0 0
- joint shoulder_pan_joint: origin xyz=0.03265 0 0.72601 rpy=0 0 0 -> xyz=0.119525 0 0.34858 rpy=0 0 0; parent arm_mount_link -> torso_lift_link
- joint upperarm_roll_joint: axis 0 0 1 -> 1 0 0
- joint wrist_flex_joint: axis 0 0 1 -> 0 1 0
- joint wrist_roll_joint: axis 0 0 1 -> 1 0 0
